File: lfo.kicad_sch (KiCad schematic)
At the start: 36 parts, among them J1 PJ398SM-12 (Tri), J2 PJ398SM-12 (square), J3 PJ398SM-12 (weird), J4 Conn_02x05_Odd_Even, Q1 BC547, SW1 SW_SPDT, U1 TL084

Commit message: successcive editing
Parts:
- removed C6: 100nFC, Capacitor_THT:C_Disc_D9.0mm_W2.5mm_P5.00mm, symbol Device:C
- D3: footprint Diode_THT:D_DO-41_SOD81_P10.16mm_Horizontal -> Diode_THT:D_DO-201AD_P3.81mm_Vertical_AnodeUp
Changed lines of the file:
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@@
 	)
 	(junction
-		(at 53.34 85.09)
+		(at 55.88 184.15)
 		(diameter 0)
 		(color 0 0 0 0)
 	)
 	(junction
-		(at 55.88 184.15)
+		(at 24.13 176.53)
 		(diameter 0)
 		(color 0 0 0 0)
 	)
 	(junction
-		(at 24.13 176.53)
+		(at 53.34 67.31)
 		(diameter 0)
 		(color 0 0 0 0)
 	)
 	(junction
-		(at 53.34 67.31)
+		(at 53.34 85.09)
 		(diameter 0)
 		(color 0 0 0 0)
@@
 	(wire
 		(pts
-			(xy 53.34 85.09) (xy 69.85 85.09)
-		)
-		(stroke
-			(width 0)
-			(type default)
-		)
-	)
-	(wire
-		(pts
 			(xy 24.13 182.88) (xy 36.83 182.88)
 		)
@@
 	(wire
 		(pts
+			(xy 53.34 85.09) (xy 69.85 85.09)
+		)
+		(stroke
+			(width 0)
+			(type default)
+		)
+	)
+	(wire
+		(pts
 			(xy 101.6 69.85) (xy 109.22 69.85)
 		)
@@
 	)
 	(symbol
-		(lib_id "Device:C")
-		(at 248.92 24.13 0)
-		(unit 1)
-		(exclude_from_sim no)
-		(in_bom yes)
-		(on_board yes)
-		(dnp no)
-		(fields_autoplaced yes)
-		(property "Reference" "C6"
-			(at 252.73 22.8599 0)
-			(effects
-				(font
-					(size 1.27 1.27)
-				)
-				(justify left)
-			)
-		)
-		(property "Value" "100nFC"
-			(at 252.73 25.3999 0)
-			(effects
-				(font
-					(size 1.27 1.27)
-				)
-				(justify left)
-			)
-		)
-		(property "Footprint" "Capacitor_THT:C_Disc_D9.0mm_W2.5mm_P5.00mm"
-			(at 249.8852 27.94 0)
-			(effects
-				(font
-					(size 1.27 1.27)
-				)
-				(hide yes)
-			)
-		)
-		(property "Datasheet" "~"
-			(at 248.92 24.13 0)
-			(effects
-				(font
-					(size 1.27 1.27)
-				)
-				(hide yes)
-			)
-		)
-		(property "Description" ""
-			(at 248.92 24.13 0)
-			(effects
-				(font
-					(size 1.27 1.27)
-				)
-			)
-		)
-		(pin "1"
-		)
-		(pin "2"
-		)
-		(instances
-			(project ""
-				(path "/b92c6e1c-e1cf-44ca-9819-a132a581d6b6"
-					(reference "C6")
-					(unit 1)
-				)
-			)
-		)
-	)
-	(symbol
 		(lib_id "Device:C_Polarized")
 		(at 55.88 180.34 0)
@@
 			)
 		)
-		(property "Footprint" "Diode_THT:D_DO-41_SOD81_P10.16mm_Horizontal"
+		(property "Footprint" "Diode_THT:D_DO-201AD_P3.81mm_Vertical_AnodeUp"
 			(at 48.26 164.465 0)
 			(effects
